File: stm32f401_devboard.rev2/stm32f401_devboard.kicad_pcb (KiCad board)
At the start: 4 copper layers, 50 x 50 mm, 31 parts, among them CON1 CORTEX-DEBUGGER, J1 USB_C, J2 Conn_02x12_Odd_Even, J5 Conn_02x12_Odd_Even, SW1 SW_Push, SW2 SW_Push, SW3 SW_Push, U1 STM32F401CCUx, U2 LM1117-3.3, Y1 12MHz, Y2 32.768K

Commit message: rev3
Parts:
- moved SW1 30.6 mm to (143.9, 103.5)
- moved C6 30.3 mm to (138.7, 103.5)
- moved C5 3.39 mm to (135.2, 100.0)
- moved C4 3.29 mm to (135.3, 97.4)
- moved Y2 3.28 mm to (133.0, 98.7)
- moved C1 2.90 mm to (136.4, 94.8)
- moved Y1 2.50 mm to (133.9, 94.2)
- moved C2 2.44 mm to (134.0, 91.2)
- moved L1 2.40 mm to (131.5, 87.8)
- moved CON1 2.40 mm to (104.0, 111.3), turned to 0 degrees
- moved R6 2.33 mm to (131.5, 90.4), turned to 90 degrees
- moved R5 0.54 mm to (130.8, 99.0)
- moved D3 0.51 mm to (129.9, 101.2)
- moved J1 0.50 mm to (104.2, 95.5)
Connections:
- J1 pad A6: PA11 -> PA12
- J1 pad A7: PA12 -> PA11
- J1 pad B6: PA11 -> PA12
- J1 pad B7: PA12 -> PA11
Routing:
- net PA14: track 46.9 -> 56.7 mm
- net PB3: track 52.2 -> 43.6 mm, vias 1 -> 2
- net PA13: track 41.0 -> 49.0 mm
- net PA9: track 72.5 -> 80.2 mm, vias 1 -> 2
- net PA10: track 74.5 -> 79.1 mm, vias 0 -> 1
- net PA12: track 42.5 -> 39.1 mm, vias 0 -> 2
- net PC15: track 10.6 -> 7.29 mm
- net PC14: track 11.9 -> 8.72 mm
- net PA11: track 38.2 -> 35.1 mm, vias 2 -> 0
- net PH0: track 12.0 -> 8.96 mm
- net PH1: track 9.85 -> 7.14 mm
- net GND: track 153.1 -> 151.3 mm, vias 16 -> 15
- net Net-(R6-Pad1): track 2.47 -> 3.83 mm
- net Net-(L1-Pad2): track 1.79 -> 1.27 mm
- net +BATT: track 28.4 -> 28.2 mm, vias 2 -> 0
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