File: stm32f401_devboard.rev2/stm32f401ccu6.sch (KiCad schematic (older format))
At the start: 29 parts, among them CON1 CORTEX-DEBUGGER, J1 USB_C, SW1 SW_Push, SW2 SW_Push, SW3 SW_Push, U1 STM32F401CCUx, U2 LM1117-3.3, Y1 12MHz, Y2 32.768K

Commit message: rev3
Parts:
- R6: value 10k -> 0
Connections:
- net PA11: now also J1.A7 (D-), J1.B7 (D-); no longer J1.A6 (D+), J1.B6 (D+)
- net PA12: now also J1.A6 (D+), J1.B6 (D+); no longer J1.A7 (D-), J1.B7 (D-)
Changed lines of the file:
@@
 	1500 1850 1450 1850
 Text GLabel 1500 2150 2    50   Input ~ 0
+PA12
+Text GLabel 1500 1850 2    50   Input ~ 0
 PA11
-Text GLabel 1500 1850 2    50   Input ~ 0
-PA12
 $Comp
 L Regulator_Linear:LM1117-3.3 U2
@@
 P 4600 2900
 F 0 "R6" H 4600 2850 50  0000 C CNN
-F 1 "10k" H 4800 2850 60  0000 C CNN
+F 1 "0" H 4800 2850 60  0000 C CNN
 F 2 "Resistor_SMD:R_0402_1005Metric" H 4600 2490 60  0001 L CNN
 F 3 "" H 4600 2400 60  0001 L CNN
