File: stm32f401_devboard/stm32f401_devboard.kicad_pcb (KiCad board)
At the start: 2 copper layers, 53 x 21 mm, 31 parts, among them CON1 CORTEX-DEBUGGER, J1 microusb, J3 Conn_01x20, J4 Conn_01x20, U1 STM32F401CCUx, U2 LM1117-3.3, Y1 12MHz, Y2 32.768K

Commit message: usb fix
Parts:
- renumbered RST to SW1, PA0 to SW2, BOOT0 to SW3
Connections:
- J1 pad 2: PA12 -> PA11
- J1 pad 3: PA11 -> PA12
- J1 pad 4: Net-(J1-Pad4) -> (no net)
Routing:
- net PA12: track 28.7 -> 29.6 mm
- net PA11: track 29.2 -> 30.1 mm
